Commit message: getting joints moving

File: client/robot.urdf (robot description, URDF)
Before this commit: robot henry2, 26 links, 25 joints
Joints:
- removed joint climber1-climber2
- removed joint climber2-climber3
- removed joint climber3-hinge5
- removed joint driveBase-hinge1
- removed joint driveBase-hinge3
- removed joint piston1-pistonArm1
- removed joint rollerhinge1-roller
- removed joint shaft1-wheel1
- removed joint shaft1-wheel2
- removed joint shaft2-wheel3
- removed joint shaft2-wheel4
- added joint climber1Climber2: type prismatic, parent climber1, child climber2, origin xyz=0 0 1.25, axis 0 0 1, limit lower=-0.75 upper=0
- added joint climber2Climber3: type prismatic, parent climber2, child climber3, origin xyz=0 0 0.75, axis 0 0 1, limit lower=-0.375 upper=0
- added joint climber3Hinge5: type revolute, parent climber3, child hinge5, origin xyz= 0 0 0.38 rpy=0 1.57 1.57, axis 0 0 1, limit lower=-1.57 upper=0
- added joint driveBaseHinge1: type revolute, parent driveBase, child hinge1, origin xyz=1.05 1.4 0.3, axis 1 0 0, limit lower=0 upper=1.57
- added joint driveBaseHinge3: type revolute, parent driveBase, child hinge3, origin xyz=1.05 0 0.35, axis 1 0 0, limit lower=0 upper=0.52
- added joint piston1PistonArm1: type prismatic, parent piston1, child pistonArm1, origin xyz=0 0 -1.075, axis 0 0 1, limit lower=-0.05 upper=0.59
- added joint rollerhinge1Roller: type continuous, parent rollerhinge1, child roller, origin xyz=-0.95 0 0 rpy=0 1.57 0, axis 0 0 1
- added joint shaft1Wheel1: type continuous, parent shaft1, child wheel1, origin xyz=0 0 1.375, axis 0 0 1
- added joint shaft1Wheel2: type continuous, parent shaft1, child wheel2, origin xyz=0 0 -1.375, axis 0 0 1
- added joint shaft2Wheel3: type continuous, parent shaft2, child wheel3, origin xyz=0 0 1.375, axis 0 0 1
- added joint shaft2Wheel4: type continuous, parent shaft2, child wheel4, origin xyz=0 0 -1.375, axis 0 0 1
